Commit message: Added a basic test rover to use in place of real thing for now

File: ros_ws/src/simulation/urdf/rover/rover.urdf.xacro (robot description, xacro)
@@ -1,3 +1,7 @@
 <?xml version="1.0"?>
+<!--
+NOTE THIS MODEL IS BROKEN RIGHT NOW
+This needs to get fixed eventually...
+-->
 <robot xmlns:xacro="http://www.ros.org/wiki/xacro" name="rover">
     <!-- IMPORTS -->

File: ros_ws/src/simulation/urdf/util/materials.xacro (robot description, xacro)
@@ -53,3 +53,13 @@
         />
     </xacro:macro>
+    <xacro:macro name = "material_gray">
+        <material name = "grey">
+            <color rgba="0.5 0.5 0.5 1.0"/>
+        </material>
+    </xacro:macro>
+    <xacro:macro name = "material_red">
+        <material name = "red">
+            <color rgba="1.0 0.0 0.0 1.0"/>
+        </material>
+    </xacro:macro>
 </robot>
