Commit message: Add missing weights to rover

File: Unity/WRover_27_Sim/Assets/Robots/wrover/wrover_27_unity.urdf (robot description, URDF)
Before this commit: robot wrover_27_simple, 17 links, 16 joints
Links:
- link base_link: mass 10.048 -> 14.6904961
- link rocker_left: mass 3.08663932 -> 3.6869132
- link rocker_right: mass 3.08663932 -> 3.6869132
- link steer_fl: mass 0.62 -> 1.00017118
- link steer_fr: mass 0.62 -> 1.00017118
- link steer_rl: mass 0.62 -> 1.00017118
- link steer_rr: mass 0.62 -> 1.00017118
